Commit message: modified gazebo.urdf

File: src/agibot_x2_pkg/urdf/x2_hand_gazebo.urdf (robot description, URDF)
Before this commit: robot x2_t2.5, 35 links, 34 joints
Links:
- link head_pitch_link: geometry collision cylinder length=0.1 radius=0.074; visual mesh filename=package://agibot_x2_pkg/meshes/head_pitch_link.STL
- link head_yaw_link: geometry collision mesh filename=package://agibot_x2_pkg/meshes/head_yaw_link.STL; visual mesh filename=package://agibot_x2_pkg/meshes/head_yaw_link.STL
- link imu_in_head_link: geometry visual mesh filename=package://agibot_x2_pkg/meshes/imu_in_head_link.STL
- link imu_in_pelvis_link: geometry visual mesh filename=package://agibot_x2_pkg/meshes/imu_in_pelvis_link.STL
- link imu_in_torso_link: geometry visual mesh filename=package://agibot_x2_pkg/meshes/imu_in_torso_link.STL
- link left_ankle_pitch_link: geometry collision mesh filename=package://agibot_x2_pkg/meshes/left_ankle_pitch_link.STL; visual mesh filename=package://agibot_x2_pkg/meshes/left_ankle_pitch_link.STL
- link left_ankle_roll_link: geometry collision mesh filename=package://agibot_x2_pkg/meshes/left_ankle_roll_link.STL; visual mesh filename=package://agibot_x2_pkg/meshes/left_ankle_roll_link.STL
- link left_elbow_link: geometry collision mesh filename=package://agibot_x2_pkg/meshes/left_elbow_link.STL; visual mesh filename=package://agibot_x2_pkg/meshes/left_elbow_link.STL
- link left_hip_pitch_link: geometry collision mesh filename=package://agibot_x2_pkg/meshes/left_hip_pitch_link.STL; visual mesh filename=package://agibot_x2_pkg/meshes/left_hip_pitch_link.STL
- link left_hip_roll_link: geometry collision mesh filename=package://agibot_x2_pkg/meshes/left_hip_roll_link.STL scale=1.0 0.9 1.0; visual mesh filename=package://agibot_x2_pkg/meshes/left_hip_roll_link.STL
- link left_hip_yaw_link: geometry collision mesh filename=package://agibot_x2_pkg/meshes/left_hip_yaw_link.STL; visual mesh filename=package://agibot_x2_pkg/meshes/left_hip_yaw_link.STL
- link left_knee_link: geometry collision mesh filename=package://agibot_x2_pkg/meshes/left_knee_link.STL; visual mesh filename=package://agibot_x2_pkg/meshes/left_knee_link.STL
- link left_shoulder_pitch_link: geometry collision mesh filename=package://agibot_x2_pkg/meshes/left_shoulder_pitch_link.STL; visual mesh filename=package://agibot_x2_pkg/meshes/left_shoulder_pitch_link.STL
- link left_shoulder_roll_link: geometry collision mesh filename=package://agibot_x2_pkg/meshes/left_shoulder_roll_link.STL; visual mesh filename=package://agibot_x2_pkg/meshes/left_shoulder_roll_link.STL
- link left_shoulder_yaw_link: geometry collision mesh filename=package://agibot_x2_pkg/meshes/left_shoulder_yaw_link.STL; visual mesh filename=package://agibot_x2_pkg/meshes/left_shoulder_yaw_link.STL
- link left_wrist_yaw_link: geometry collision mesh filename=package://agibot_x2_pkg/meshes/left_wrist_hand_link.STL; visual mesh filename=package://agibot_x2_pkg/meshes/left_wrist_hand_link.STL
- link pelvis: geometry collision mesh filename=package://agibot_x2_pkg/meshes/pelvis.STL; visual mesh filename=package://agibot_x2_pkg/meshes/pelvis.STL
- link rgb_head_center_link: geometry visual mesh filename=package://agibot_x2_pkg/meshes/rgb_head_center_link.STL
- link rgb_head_rear_link: geometry visual mesh filename=package://agibot_x2_pkg/meshes/rgb_head_rear_link.STL
- link rgbd_head_front_link: geometry visual mesh filename=package://agibot_x2_pkg/meshes/rgbd_head_front_link.STL
- link right_ankle_pitch_link: geometry collision mesh filename=package://agibot_x2_pkg/meshes/right_ankle_pitch_link.STL; visual mesh filename=package://agibot_x2_pkg/meshes/right_ankle_pitch_link.STL
- link right_ankle_roll_link: geometry collision mesh filename=package://agibot_x2_pkg/meshes/right_ankle_roll_link.STL; visual mesh filename=package://agibot_x2_pkg/meshes/right_ankle_roll_link.STL
- link right_elbow_link: geometry collision mesh filename=package://agibot_x2_pkg/meshes/right_elbow_link.STL; visual mesh filename=package://agibot_x2_pkg/meshes/right_elbow_link.STL
- link right_hip_pitch_link: geometry collision mesh filename=package://agibot_x2_pkg/meshes/right_hip_pitch_link.STL; visual mesh filename=package://agibot_x2_pkg/meshes/right_hip_pitch_link.STL
- link right_hip_roll_link: geometry collision mesh filename=package://agibot_x2_pkg/meshes/right_hip_roll_link.STL scale=1.0 0.9 1.0; visual mesh filename=package://agibot_x2_pkg/meshes/right_hip_roll_link.STL
- link right_hip_yaw_link: geometry collision mesh filename=package://agibot_x2_pkg/meshes/right_hip_yaw_link.STL; visual mesh filename=package://agibot_x2_pkg/meshes/right_hip_yaw_link.STL
- link right_knee_link: geometry collision mesh filename=package://agibot_x2_pkg/meshes/right_knee_link.STL; visual mesh filename=package://agibot_x2_pkg/meshes/right_knee_link.STL
- link right_shoulder_pitch_link: geometry collision mesh filename=package://agibot_x2_pkg/meshes/right_shoulder_pitch_link.STL; visual mesh filename=package://agibot_x2_pkg/meshes/right_shoulder_pitch_link.STL
- link right_shoulder_roll_link: geometry collision mesh filename=package://agibot_x2_pkg/meshes/right_shoulder_roll_link.STL; visual mesh filename=package://agibot_x2_pkg/meshes/right_shoulder_roll_link.STL
- link right_shoulder_yaw_link: geometry collision mesh filename=package://agibot_x2_pkg/meshes/right_shoulder_yaw_link.STL; visual mesh filename=package://agibot_x2_pkg/meshes/right_shoulder_yaw_link.STL
- link right_wrist_yaw_link: geometry collision mesh filename=package://agibot_x2_pkg/meshes/right_wrist_hand_link.STL; visual mesh filename=package://agibot_x2_pkg/meshes/right_wrist_hand_link.STL
- link stereo_head_front_link: geometry visual mesh filename=package://agibot_x2_pkg/meshes/stereo_head_front_link.STL
- link torso_link: geometry collision mesh filename=package://agibot_x2_pkg/meshes/torso_plus_link.STL; visual mesh filename=package://agibot_x2_pkg/meshes/torso_plus_link.STL
- link waist_pitch_link: geometry visual mesh filename=package://agibot_x2_pkg/meshes/waist_pitch_link.STL
- link waist_yaw_link: geometry visual mesh filename=package://agibot_x2_pkg/meshes/waist_yaw_link.STL

Commit message: update gazebo.urdf

File: src/agibot_x2_pkg/urdf/x2_hand_gazebo.urdf (robot description, URDF)
Before this commit: robot x2_t2.5, 35 links, 34 joints
Links:
- link head_pitch_link: geometry collision cylinder length=0.1 radius=0.074; visual mesh filename=file:///home/utente/Desktop/SmartRobotics/install/agibot_x2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
- link head_yaw_link: geometry collision mesh filename=file:///home/utente/Desktop/SmartRobotics/install/agibot_x2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; visual mesh filename=file:///home/utente/Desktop/SmartRobotics/install/agibot_x2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
- link imu_in_head_link: geometry visual mesh filename=file:///home/utente/Desktop/SmartRobotics/install/agibot_x2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
- link imu_in_pelvis_link: geometry visual mesh filename=file:///home/utente/Desktop/SmartRobotics/install/agibot_x2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
- link imu_in_torso_link: geometry visual mesh filename=file:///home/utente/Desktop/SmartRobotics/install/agibot_x2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
- link left_ankle_pitch_link: geometry collision mesh filename=file:///home/utente/Desktop/SmartRobotics/install/agibot_x2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; visual mesh filename=file:///home/utente/Desktop/SmartRobotics/install/agibot_x2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
- link left_ankle_roll_link: geometry collision mesh filename=file:///home/utente/Desktop/SmartRobotics/install/agibot_x2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; visual mesh filename=file:///home/utente/Desktop/SmartRobotics/install/agibot_x2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
- link left_elbow_link: geometry collision mesh filename=file:///home/utente/Desktop/SmartRobotics/install/agibot_x2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; visual mesh filename=file:///home/utente/Desktop/SmartRobotics/install/agibot_x2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
- link left_hip_pitch_link: geometry collision mesh filename=file:///home/utente/Desktop/SmartRobotics/install/agibot_x2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; visual mesh filename=file:///home/utente/Desktop/SmartRobotics/install/agibot_x2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
- link left_hip_roll_link: geometry collision mesh filename=file:///home/utente/Desktop/SmartRobotics/install/agibot_x2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 scale=1.0 0.9 1.0; visual mesh filename=file:///home/utente/Desktop/SmartRobotics/install/agibot_x2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
- link left_hip_yaw_link: geometry collision mesh filename=file:///home/utente/Desktop/SmartRobotics/install/agibot_x2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; visual mesh filename=file:///home/utente/Desktop/SmartRobotics/install/agibot_x2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
- link left_knee_link: geometry collision mesh filename=file:///home/utente/Desktop/SmartRobotics/install/agibot_x2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; visual mesh filename=file:///home/utente/Desktop/SmartRobotics/install/agibot_x2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
- link left_shoulder_pitch_link: geometry collision mesh filename=file:///home/utente/Desktop/SmartRobotics/install/agibot_x2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; visual mesh filename=file:///home/utente/Desktop/SmartRobotics/install/agibot_x2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
- link left_shoulder_roll_link: geometry collision mesh filename=file:///home/utente/Desktop/SmartRobotics/install/agibot_x2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; visual mesh filename=file:///home/utente/Desktop/SmartRobotics/install/agibot_x2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
- link left_shoulder_yaw_link: geometry collision mesh filename=file:///home/utente/Desktop/SmartRobotics/install/agibot_x2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; visual mesh filename=file:///home/utente/Desktop/SmartRobotics/install/agibot_x2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
- link left_wrist_yaw_link: geometry collision mesh filename=file:///home/utente/Desktop/SmartRobotics/install/agibot_x2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; visual mesh filename=file:///home/utente/Desktop/SmartRobotics/install/agibot_x2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
- link pelvis: geometry collision mesh filename=file:///home/utente/Desktop/SmartRobotics/install/agibot_x2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; visual mesh filename=file:///home/utente/Desktop/SmartRobotics/install/agibot_x2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
- link rgb_head_center_link: geometry visual mesh filename=file:///home/utente/Desktop/SmartRobotics/install/agibot_x2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
- link rgb_head_rear_link: geometry visual mesh filename=file:///home/utente/Desktop/SmartRobotics/install/agibot_x2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
- link rgbd_head_front_link: geometry visual mesh filename=file:///home/utente/Desktop/SmartRobotics/install/agibot_x2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
- link right_ankle_pitch_link: geometry collision mesh filename=file:///home/utente/Desktop/SmartRobotics/install/agibot_x2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; visual mesh filename=file:///home/utente/Desktop/SmartRobotics/install/agibot_x2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
- link right_ankle_roll_link: geometry collision mesh filename=file:///home/utente/Desktop/SmartRobotics/install/agibot_x2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; visual mesh filename=file:///home/utente/Desktop/SmartRobotics/install/agibot_x2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
- link right_elbow_link: geometry collision mesh filename=file:///home/utente/Desktop/SmartRobotics/install/agibot_x2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; visual mesh filename=file:///home/utente/Desktop/SmartRobotics/install/agibot_x2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
- link right_hip_pitch_link: geometry collision mesh filename=file:///home/utente/Desktop/SmartRobotics/install/agibot_x2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; visual mesh filename=file:///home/utente/Desktop/SmartRobotics/install/agibot_x2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
- link right_hip_roll_link: geometry collision mesh filename=file:///home/utente/Desktop/SmartRobotics/install/agibot_x2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 scale=1.0 0.9 1.0; visual mesh filename=file:///home/utente/Desktop/SmartRobotics/install/agibot_x2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
- link right_hip_yaw_link: geometry collision mesh filename=file:///home/utente/Desktop/SmartRobotics/install/agibot_x2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; visual mesh filename=file:///home/utente/Desktop/SmartRobotics/install/agibot_x2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
- link right_knee_link: geometry collision mesh filename=file:///home/utente/Desktop/SmartRobotics/install/agibot_x2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; visual mesh filename=file:///home/utente/Desktop/SmartRobotics/install/agibot_x2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
- link right_shoulder_pitch_link: geometry collision mesh filename=file:///home/utente/Desktop/SmartRobotics/install/agibot_x2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; visual mesh filename=file:///home/utente/Desktop/SmartRobotics/install/agibot_x2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
- link right_shoulder_roll_link: geometry collision mesh filename=file:///home/utente/Desktop/SmartRobotics/install/agibot_x2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; visual mesh filename=file:///home/utente/Desktop/SmartRobotics/install/agibot_x2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
- link right_shoulder_yaw_link: geometry collision mesh filename=file:///home/utente/Desktop/SmartRobotics/install/agibot_x2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; visual mesh filename=file:///home/utente/Desktop/SmartRobotics/install/agibot_x2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
- link right_wrist_yaw_link: geometry collision mesh filename=file:///home/utente/Desktop/SmartRobotics/install/agibot_x2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; visual mesh filename=file:///home/utente/Desktop/SmartRobotics/install/agibot_x2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
- link stereo_head_front_link: geometry visual mesh filename=file:///home/utente/Desktop/SmartRobotics/install/agibot_x2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
- link torso_link: geometry collision mesh filename=file:///home/utente/Desktop/SmartRobotics/install/agibot_x2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; visual mesh filename=file:///home/utente/Desktop/SmartRobotics/install/agibot_x2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
- link waist_pitch_link: geometry visual mesh filename=file:///home/utente/Desktop/SmartRobotics/install/agibot_x2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
- link waist_yaw_link: geometry visual mesh filename=file:///home/utente/Desktop/SmartRobotics/install/agibot_x2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
