Commit message: Fixed gaz resources and movement script

File: src/agibot_x2_pkg/urdf/x2_hand_gazebo.urdf (robot description, URDF)
Before this commit: robot x2_t2.5, 35 links, 34 joints
Links:
- link head_yaw_link: geometry collision cylinder length=0.06 radius=0.035; visual mesh filename=package://agibot_x2_pkg/meshes/head_yaw_link.STL
- link left_ankle_pitch_link: geometry collision cylinder length=0.06 radius=0.035; visual mesh filename=package://agibot_x2_pkg/meshes/left_ankle_pitch_link.STL
- link left_ankle_roll_link: geometry collision box size=0.20 0.10 0.04; visual mesh filename=package://agibot_x2_pkg/meshes/left_ankle_roll_link.STL
- link left_elbow_link: geometry collision cylinder length=0.12 radius=0.03; visual mesh filename=package://agibot_x2_pkg/meshes/left_elbow_link.STL
- link left_hip_pitch_link: geometry collision cylinder length=0.08 radius=0.06; visual mesh filename=package://agibot_x2_pkg/meshes/left_hip_pitch_link.STL
- link left_hip_roll_link: geometry collision cylinder length=0.12 radius=0.05; visual mesh filename=package://agibot_x2_pkg/meshes/left_hip_roll_link.STL
- link left_hip_yaw_link: geometry collision cylinder length=0.18 radius=0.05; visual mesh filename=package://agibot_x2_pkg/meshes/left_hip_yaw_link.STL
- link left_knee_link: geometry collision cylinder length=0.24 radius=0.045; visual mesh filename=package://agibot_x2_pkg/meshes/left_knee_link.STL
- link left_shoulder_pitch_link: geometry collision cylinder length=0.08 radius=0.04; visual mesh filename=package://agibot_x2_pkg/meshes/left_shoulder_pitch_link.STL
- link left_shoulder_roll_link: geometry collision cylinder length=0.10 radius=0.035; visual mesh filename=package://agibot_x2_pkg/meshes/left_shoulder_roll_link.STL
- link left_shoulder_yaw_link: geometry collision cylinder length=0.10 radius=0.035; visual mesh filename=package://agibot_x2_pkg/meshes/left_shoulder_yaw_link.STL
- link left_wrist_yaw_link: geometry collision box size=0.06 0.08 0.12; visual mesh filename=package://agibot_x2_pkg/meshes/left_wrist_hand_link.STL
- link pelvis: geometry collision box size=0.20 0.26 0.16; visual mesh filename=package://agibot_x2_pkg/meshes/pelvis.STL
- link right_ankle_pitch_link: geometry collision cylinder length=0.06 radius=0.035; visual mesh filename=package://agibot_x2_pkg/meshes/right_ankle_pitch_link.STL
- link right_ankle_roll_link: geometry collision box size=0.20 0.10 0.04; visual mesh filename=package://agibot_x2_pkg/meshes/right_ankle_roll_link.STL
- link right_elbow_link: geometry collision cylinder length=0.12 radius=0.03; visual mesh filename=package://agibot_x2_pkg/meshes/right_elbow_link.STL
- link right_hip_pitch_link: geometry collision cylinder length=0.08 radius=0.06; visual mesh filename=package://agibot_x2_pkg/meshes/right_hip_pitch_link.STL
- link right_hip_roll_link: geometry collision cylinder length=0.12 radius=0.05; visual mesh filename=package://agibot_x2_pkg/meshes/right_hip_roll_link.STL
- link right_hip_yaw_link: geometry collision cylinder length=0.18 radius=0.05; visual mesh filename=package://agibot_x2_pkg/meshes/right_hip_yaw_link.STL
- link right_knee_link: geometry collision cylinder length=0.24 radius=0.045; visual mesh filename=package://agibot_x2_pkg/meshes/right_knee_link.STL
- link right_shoulder_pitch_link: geometry collision cylinder length=0.08 radius=0.04; visual mesh filename=package://agibot_x2_pkg/meshes/right_shoulder_pitch_link.STL
- link right_shoulder_roll_link: geometry collision cylinder length=0.10 radius=0.035; visual mesh filename=package://agibot_x2_pkg/meshes/right_shoulder_roll_link.STL
- link right_shoulder_yaw_link: geometry collision cylinder length=0.10 radius=0.035; visual mesh filename=package://agibot_x2_pkg/meshes/right_shoulder_yaw_link.STL
- link right_wrist_yaw_link: geometry collision box size=0.06 0.08 0.12; visual mesh filename=package://agibot_x2_pkg/meshes/right_wrist_hand_link.STL
- link torso_link: geometry collision box size=0.22 0.32 0.40; visual mesh filename=package://agibot_x2_pkg/meshes/torso_plus_link.STL

Commit message: commit pre-pull

File: src/agibot_x2_pkg/urdf/x2_hand_gazebo.urdf (robot description, URDF)
Before this commit: robot x2_t2.5, 42 links, 41 joints
Links:
- added link left_tcp_link, mass 1.0e-03; collision box size=0.01 0.01 0.01; visual box size=0.01 0.01 0.01
- added link right_tcp_link, mass 1.0e-03; collision box size=0.01 0.01 0.01; visual box size=0.01 0.01 0.01
Joints:
- added joint left_tcp_joint: type fixed, parent left_gripper_base_link, child left_tcp_link, origin xyz=0.0 0.0 -0.045 rpy=0 0 0
- added joint right_tcp_joint: type fixed, parent right_gripper_base_link, child right_tcp_link, origin xyz=0.0 0.0 -0.045 rpy=0 0 0
- joint left_gripper_left_finger_joint: origin xyz=0.0 0.01 -0.045 -> xyz=0.0 0.02 -0.045
- joint left_gripper_right_finger_joint: origin xyz=0.0 -0.01 -0.045 -> xyz=0.0 -0.02 -0.045
- joint right_gripper_left_finger_joint: origin xyz=0.0 0.01 -0.045 -> xyz=0.0 0.02 -0.045
- joint right_gripper_right_finger_joint: origin xyz=0.0 -0.01 -0.045 -> xyz=0.0 -0.02 -0.045

Commit message: Other fixes

File: src/agibot_x2_pkg/urdf/x2_hand_gazebo.urdf (robot description, URDF)
Before this commit: robot x2_t2.5, 44 links, 43 joints
Joints:
- joint left_tcp_joint: origin xyz=0.0 0.0 -0.045 rpy=0 0 0 -> xyz=0.0 0.0 -0.075 rpy=0 0 0
- joint right_tcp_joint: origin xyz=0.0 0.0 -0.045 rpy=0 0 0 -> xyz=0.0 0.0 -0.075 rpy=0 0 0

Commit message: Added moveit framework (only table as obstacle and right_hand as cosa da muovere), fixed some stuff for warnings

File: src/agibot_x2_pkg/urdf/x2_hand_gazebo.urdf (robot description, URDF)
Before this commit: robot x2_t2.5, 48 links, 47 joints
Links:
- link imu_in_head_link: geometry collision box size=0.001 0.001 0.001; visual mesh filename=package://agibot_x2_pkg/meshes/imu_in_head_link.STL
- link imu_in_pelvis_link: geometry collision box size=0.001 0.001 0.001; visual mesh filename=package://agibot_x2_pkg/meshes/imu_in_pelvis_link.STL
- link imu_in_torso_link: geometry collision box size=0.001 0.001 0.001; visual mesh filename=package://agibot_x2_pkg/meshes/imu_in_torso_link.STL
- link left_tcp_link: geometry collision box size=0.001 0.001 0.001; visual box size=0.01 0.01 0.01
- link rgb_head_center_link: geometry collision box size=0.001 0.001 0.001; visual mesh filename=package://agibot_x2_pkg/meshes/rgb_head_center_link.STL
- link rgb_head_rear_link: geometry collision box size=0.001 0.001 0.001; visual mesh filename=package://agibot_x2_pkg/meshes/rgb_head_rear_link.STL
- link rgbd_head_front_link: geometry collision box size=0.001 0.001 0.001; visual mesh filename=package://agibot_x2_pkg/meshes/rgbd_head_front_link.STL
- link right_gripper_camera_link: geometry collision box size=0.001 0.001 0.001; visual box size=0.008 0.008 0.008
- link right_tcp_link: geometry collision box size=0.001 0.001 0.001; visual box size=0.01 0.01 0.01
- link stereo_head_front_link: geometry collision box size=0.001 0.001 0.001; visual mesh filename=package://agibot_x2_pkg/meshes/stereo_head_front_link.STL
- link waist_pitch_link: geometry collision box size=0.001 0.001 0.001; visual mesh filename=package://agibot_x2_pkg/meshes/waist_pitch_link.STL
- link waist_yaw_link: geometry collision box size=0.001 0.001 0.001; visual mesh filename=package://agibot_x2_pkg/meshes/waist_yaw_link.STL

Commit message: backup

File: src/agibot_x2_pkg/urdf/x2_hand_gazebo.urdf (robot description, URDF)
Before this commit: robot x2_t2.5, 48 links, 47 joints
Links:
- added link left_gripper_camera_link, mass 0.001; visual box size=0.008 0.008 0.008
Joints:
- added joint left_gripper_camera_joint: type fixed, parent left_gripper_base_link, child left_gripper_camera_link, origin xyz=0 0 -0.005 rpy=0 1.5707963 0

Commit message: Merge and fix robot movements

File: src/agibot_x2_pkg/urdf/x2_hand_gazebo.urdf (robot description, URDF)
Before this commit: robot agibot_x2, 49 links, 48 joints
Links:
- link left_tcp_link: geometry visual box size=0.01 0.01 0.01
- link right_tcp_link: geometry visual box size=0.01 0.01 0.01
