Commit message: Sostituito gripper

File: src/agibot_x2_pkg/urdf/OLD_WORKING_x2_hand_gazebo.urdf (robot description, URDF)
Before this commit: robot x2_t2.5, 42 links, 41 joints
Links:
- link left_gripper_base_link: mass 0.1 -> 0.05; geometry collision box size=0.05 0.05 0.02; visual mesh filename=package://agibot_x2_pkg/meshes/gripper/gripper_base.STL
- link left_gripper_left_finger_link: mass 0.1 -> 0.02; geometry collision box size=0.006 0.05 0.10; visual mesh filename=package://agibot_x2_pkg/meshes/gripper/gripper_finger.STL
- link left_gripper_right_finger_link: mass 0.1 -> 0.02; geometry collision box size=0.006 0.05 0.10; visual mesh filename=package://agibot_x2_pkg/meshes/gripper/gripper_finger.STL
- link right_gripper_base_link: mass 0.1 -> 0.05; geometry collision box size=0.05 0.05 0.02; visual mesh filename=package://agibot_x2_pkg/meshes/gripper/gripper_base.STL
- link right_gripper_left_finger_link: mass 0.1 -> 0.02; geometry collision box size=0.006 0.05 0.10; visual mesh filename=package://agibot_x2_pkg/meshes/gripper/gripper_finger.STL
- link right_gripper_right_finger_link: mass 0.1 -> 0.02; geometry collision box size=0.006 0.05 0.10; visual mesh filename=package://agibot_x2_pkg/meshes/gripper/gripper_finger.STL
Joints:
- joint left_gripper_left_finger_joint: axis 0 1 0 -> 1 0 0; limit lower=0 upper=0.04 effort=100.0 velocity=4.0 -> lower=0 upper=0.037 effort=20 velocity=0.05; origin xyz=0.0 0.01 -0.045 -> xyz=0.006 0 -0.02 rpy=0 0 0
- joint left_gripper_mount_joint: origin xyz=0.0 0 -0.01 rpy=0.0 0 0 -> xyz=0 0 0 rpy=0 0 0
- joint left_gripper_right_finger_joint: axis 0 -1 0 -> -1 0 0; limit lower=0 upper=0.04 effort=100.0 velocity=4.0 -> lower=0 upper=0.037 effort=20 velocity=0.05; origin xyz=0.0 -0.01 -0.045 -> xyz=-0.006 0 -0.02 rpy=0 0 0
- joint left_shoulder_roll_joint: origin xyz=-0.00049991072907324 0.0495 0 rpy=0 0 0 -> xyz=-0.000499991072907324 0.0495 0 rpy=0 0 0
- joint right_gripper_left_finger_joint: axis 0 1 0 -> 1 0 0; limit lower=0 upper=0.04 effort=100.0 velocity=4.0 -> lower=0 upper=0.037 effort=20 velocity=0.05; origin xyz=0.0 0.01 -0.045 -> xyz=0.006 0 -0.02 rpy=0 0 0
- joint right_gripper_mount_joint: origin xyz=0.0 0 -0.01 rpy=0.0 0 0 -> xyz=0 0 0 rpy=0 0 0
- joint right_gripper_right_finger_joint: axis 0 -1 0 -> -1 0 0; limit lower=0 upper=0.04 effort=100.0 velocity=4.0 -> lower=0 upper=0.037 effort=20 velocity=0.05; origin xyz=0.0 -0.01 -0.045 -> xyz=-0.006 0 -0.02 rpy=0 0 0
