Commit message: Cameras and env with books

File: src/agibot_x2_pkg/urdf/full_scene.urdf (robot description, URDF)
Before this commit: robot full_scene, 1 links, 0 joints
Links:
- added link table_camera_link, mass 0.001; visual box size=0.02 0.02 0.02
Joints:
- added joint table_camera_joint: type fixed, parent base_link, child table_camera_link, origin xyz=-1.05 0.80 1.55 rpy=0 1.5707963 0

File: src/agibot_x2_pkg/urdf/table.urdf (robot description, URDF)
Before this commit: robot table, 1 links, 0 joints
Links:
- added link table_camera_link, mass 0.001; visual box size=0.02 0.02 0.02
Joints:
- added joint table_camera_joint: type fixed, parent base_link, child table_camera_link, origin xyz=0 0 1.55 rpy=0 1.5707963 0

File: src/agibot_x2_pkg/urdf/x2_hand_gazebo.urdf (robot description, URDF)
Before this commit: robot x2_t2.5, 42 links, 41 joints
Links:
- added link left_gripper_camera_link, mass 0.001; visual box size=0.008 0.008 0.008
- added link right_gripper_camera_link, mass 0.001; visual box size=0.008 0.008 0.008
Joints:
- added joint left_gripper_camera_joint: type fixed, parent left_gripper_base_link, child left_gripper_camera_link, origin xyz=0 0 -0.005 rpy=0 1.5707963 0
- added joint right_gripper_camera_joint: type fixed, parent right_gripper_base_link, child right_gripper_camera_link, origin xyz=0 0 -0.005 rpy=0 1.5707963 0

Commit message: Commented cameras

File: src/agibot_x2_pkg/urdf/full_scene.urdf (robot description, URDF)
Before this commit: robot full_scene, 2 links, 1 joints
Links:
- removed link table_camera_link
Joints:
- removed joint table_camera_joint

File: src/agibot_x2_pkg/urdf/table.urdf (robot description, URDF)
Before this commit: robot table, 2 links, 1 joints
Links:
- removed link table_camera_link
Joints:
- removed joint table_camera_joint

File: src/agibot_x2_pkg/urdf/x2_hand_gazebo.urdf (robot description, URDF)
Before this commit: robot x2_t2.5, 46 links, 45 joints
Links:
- removed link left_gripper_camera_link
- removed link right_gripper_camera_link
Joints:
- removed joint left_gripper_camera_joint
- removed joint right_gripper_camera_joint
