Commit message: complete scene in Blender and scripts to detect and identify books

File: src/agibot_x2_pkg/urdf/bookshelf.urdf (robot description, URDF)
Before this commit: robot bookshelf, 1 links, 0 joints
Links:
- link base_link: geometry collision box size=0.022 0.300 1.350; collision box size=0.022 0.300 1.350

File: src/agibot_x2_pkg/urdf/x2_hand_gazebo.urdf (robot description, URDF)
Before this commit: robot x2_t2.5, 35 links, 34 joints
Links:
- added link left_gripper_base_link, mass 0.06; collision mesh filename=package://agibot_x2_pkg/meshes/gripper/gripper_base.STL; visual mesh filename=package://agibot_x2_pkg/meshes/gripper/gripper_base.STL
- added link left_gripper_left_finger_link, mass 0.036; collision mesh filename=package://agibot_x2_pkg/meshes/gripper/gripper_finger.STL; visual mesh filename=package://agibot_x2_pkg/meshes/gripper/gripper_finger.STL
- added link left_gripper_right_finger_link, mass 0.036; collision mesh filename=package://agibot_x2_pkg/meshes/gripper/gripper_finger.STL; visual mesh filename=package://agibot_x2_pkg/meshes/gripper/gripper_finger.STL
- link left_wrist_yaw_link: geometry 
Joints:
- added joint left_gripper_left_finger_joint: type prismatic, parent left_gripper_base_link, child left_gripper_left_finger_link, origin xyz=0.002 0 -0.02 rpy=0 0 0, axis 1 0 0, limit lower=0 upper=0.037 effort=20 velocity=0.05
- added joint left_gripper_mount_joint: type fixed, parent left_wrist_yaw_link, child left_gripper_base_link, origin xyz=0 0 0 rpy=0 0 0
- added joint left_gripper_right_finger_joint: type prismatic, parent left_gripper_base_link, child left_gripper_right_finger_link, origin xyz=-0.002 0 -0.02 rpy=0 0 0, axis -1 0 0, limit lower=0 upper=0.037 effort=20 velocity=0.05

Commit message: Environment con camera e prova identificazione libri

File: src/agibot_x2_pkg/urdf/bookshelf.urdf (robot description, URDF)
Before this commit: robot bookshelf, 1 links, 0 joints
Links:
- added link shelf_camera_link, mass 0.001; visual box size=0.02 0.02 0.02
Joints:
- added joint shelf_camera_joint: type fixed, parent base_link, child shelf_camera_link, origin xyz=-0.16 0.75 1.50 rpy=0 0.55 -1.5707963

File: src/agibot_x2_pkg/urdf/x2_hand_gazebo.urdf (robot description, URDF)
Before this commit: robot x2_t2.5, 44 links, 43 joints
Links:
- link left_tcp_link: geometry visual box size=0.01 0.01 0.01
- link right_tcp_link: geometry visual box size=0.01 0.01 0.01
