Commit message: Full scene and test gripper

File: src/agibot_x2_pkg/urdf/table.urdf (robot description, URDF)
Before this commit: robot table, 1 links, 0 joints
Links:
- link base_link: geometry collision box size=0.040 0.040 0.705; collision box size=0.040 0.040 0.705

File: src/agibot_x2_pkg/urdf/x2_hand_gazebo.urdf (robot description, URDF)
Before this commit: robot x2_t2.5, 35 links, 34 joints
Links:
- added link left_gripper_base_link, mass 0.05; collision box size=0.05 0.05 0.02; visual mesh filename=package://agibot_x2_pkg/meshes/gripper/gripper_base.STL
- added link left_gripper_left_finger_link, mass 0.02; collision box size=0.006 0.05 0.10; visual mesh filename=package://agibot_x2_pkg/meshes/gripper/gripper_finger.STL
- added link left_gripper_right_finger_link, mass 0.02; collision box size=0.006 0.05 0.10; visual mesh filename=package://agibot_x2_pkg/meshes/gripper/gripper_finger.STL
- added link right_gripper_base_link, mass 0.05; collision box size=0.05 0.05 0.02; visual mesh filename=package://agibot_x2_pkg/meshes/gripper/gripper_base.STL
- added link right_gripper_left_finger_link, mass 0.02; collision box size=0.006 0.05 0.10; visual mesh filename=package://agibot_x2_pkg/meshes/gripper/gripper_finger.STL
- added link right_gripper_right_finger_link, mass 0.02; collision box size=0.006 0.05 0.10; visual mesh filename=package://agibot_x2_pkg/meshes/gripper/gripper_finger.STL
- added link world
- link left_wrist_yaw_link: geometry 
- link right_wrist_yaw_link: geometry 
Joints:
- added joint left_gripper_left_finger_joint: type prismatic, parent left_gripper_base_link, child left_gripper_left_finger_link, origin xyz=0.006 0 -0.02 rpy=0 0 0, axis 1 0 0, limit lower=0 upper=0.037 effort=20 velocity=0.05
- added joint left_gripper_mount_joint: type fixed, parent left_wrist_yaw_link, child left_gripper_base_link, origin xyz=0 0 0 rpy=0 0 0
- added joint left_gripper_right_finger_joint: type prismatic, parent left_gripper_base_link, child left_gripper_right_finger_link, origin xyz=-0.006 0 -0.02 rpy=0 0 0, axis -1 0 0, limit lower=0 upper=0.037 effort=20 velocity=0.05
- added joint right_gripper_left_finger_joint: type prismatic, parent right_gripper_base_link, child right_gripper_left_finger_link, origin xyz=0.006 0 -0.02 rpy=0 0 0, axis 1 0 0, limit lower=0 upper=0.037 effort=20 velocity=0.05
- added joint right_gripper_mount_joint: type fixed, parent right_wrist_yaw_link, child right_gripper_base_link, origin xyz=0 0 0 rpy=0 0 0
- added joint right_gripper_right_finger_joint: type prismatic, parent right_gripper_base_link, child right_gripper_right_finger_link, origin xyz=-0.006 0 -0.02 rpy=0 0 0, axis -1 0 0, limit lower=0 upper=0.037 effort=20 velocity=0.05
- added joint world_to_pelvis_joint: type fixed, parent world, child pelvis, origin xyz=0 0 0 rpy=0 0 0

Commit message: test gripper and ISBN

File: src/agibot_x2_pkg/urdf/table.urdf (robot description, URDF)
Before this commit: robot table, 1 links, 0 joints
Links:
- added link table_camera_link, mass 0.001; visual box size=0.02 0.02 0.02
Joints:
- added joint table_camera_joint: type fixed, parent base_link, child table_camera_link, origin xyz=0.405 -0.11 1.30 rpy=0 1.5707963 0

Commit message: prova intera pipeline con robot che cammina

File: src/agibot_x2_pkg/urdf/table.urdf (robot description, URDF)
Before this commit: robot table, 2 links, 1 joints
Joints:
- joint table_camera_joint: origin xyz=0.405 -0.11 1.30 rpy=0 1.5707963 0 -> xyz=0.53 -0.11 1.30 rpy=0 1.5707963 0

File: src/agibot_x2_pkg/urdf/x2_hand_gazebo.urdf (robot description, URDF)
Before this commit: robot x2_t2.5, 44 links, 43 joints
Links:
- added link base_x_link, mass 0.5
- added link base_y_link, mass 0.5
- added link base_z_link, mass 0.5
- added link right_gripper_camera_link, mass 0.001; visual box size=0.008 0.008 0.008
Joints:
- removed joint world_to_pelvis_joint
- added joint base_x_joint: type prismatic, parent world, child base_x_link, origin xyz=0 0 0 rpy=0 0 0, axis 1 0 0, limit lower=-1.0 upper=5.0 effort=2000 velocity=2.0
- added joint base_y_joint: type prismatic, parent base_x_link, child base_y_link, origin xyz=0 0 0 rpy=0 0 0, axis 0 1 0, limit lower=-3.0 upper=3.0 effort=2000 velocity=2.0
- added joint base_yaw_joint: type revolute, parent base_z_link, child pelvis, origin xyz=0 0 0 rpy=0 0 0, axis 0 0 1, limit lower=-3.15 upper=3.15 effort=2000 velocity=2.0
- added joint base_z_joint: type prismatic, parent base_y_link, child base_z_link, origin xyz=0 0 0 rpy=0 0 0, axis 0 0 1, limit lower=-0.10 upper=0.50 effort=2000 velocity=1.0
- added joint right_gripper_camera_joint: type fixed, parent right_gripper_base_link, child right_gripper_camera_link, origin xyz=0 0 -0.005 rpy=0 1.5707963 0
